File: pcb/large/rcstick-f.brd (EAGLE design)
At the start: 27.6 x 43.1 mm, 41 parts, among them J1 MOLEX_48037-0001, J2 2212S, SW1 SKRPACE010, U1 STM32F042KT, U2 CC2500, U3 MCP1703AT-3302E/CB, X1 8MHz/15pF, X2 26MHz/9pF, X3 (50 Ohm)

Commit message: renumbering capacities
Parts:
- removed C26: 1.8p, gen-discrete3:RCL_C0402_HS
- removed C27: 1.5p, gen-discrete3:RCL_C0402_HS
- added C13, C14: 220p, gen-discrete3:RCL_C0402_HS
- C15, C16: value 220p -> 0.1u
- C17: value 0.1u -> 220p
- C18: value 0.1u -> 12p
- C19: value 220p -> 12p
- C20, C21: value 12p -> 100p
- C22, C23: value 100p -> 1p
- C24: value 1p -> 1.8p
- C25: value 1p -> 1.5p
- moved C19 11.7 mm to (16.1, 24.5), turned to 90 degrees
- moved C15 9.74 mm to (12.7, 25.4), flipped to the bottom
- moved C21 9.20 mm to (9.02, 30.4), turned to 0 degrees
- moved C17 8.13 mm to (4.83, 27.4), flipped to the top
- moved C20 6.33 mm to (9.02, 31.5)
- moved C16 5.37 mm to (10.2, 27.9), turned to 0 degrees
- moved C22 4.33 mm to (12.7, 29.2)
- moved C23 3.86 mm to (12.7, 31.5)
- moved C18 3.83 mm to (14.0, 27.6)
- moved C24 3.74 mm to (16.4, 29.8)
- moved C25 3.74 mm to (16.4, 32.1), turned to 180 degrees
Connections:
- net +3V3: now also C13.1, C14.1; no longer C18.1, C19.1
- net GND: now also C13.2, C14.2, C22.2, C25.2; no longer C20.2, C21.2, C26.2, C27.2
- net N$10: now also C23.2, C24.1; no longer C25.2, C26.1
- net N$11: now also C25.1; no longer C27.1
- net N$5: now also C20.2, C23.1; no longer C22.2, C25.1
- net N$9: now also C21.2, C22.1; no longer C23.2, C24.1
- net RF_N: now also C20.1; no longer C22.1
- net RF_P: now also C21.1; no longer C23.1
- net XOSC1: now also C19.1; no longer C21.1
- net XOSC2: now also C18.1; no longer C20.1

Commit message: refine wiring
Parts:
- J1: device Molex - 48037-0001:MOLEX_48037-0001_1 -> Molex-48037-0001:MOLEX_48037-0001_1
- moved LED1 18.1 mm to (2.79, 17.9), turned to 270 degrees
- moved R3 15.7 mm to (4.32, 17.9), turned to 270 degrees
Connections:
- net LED: now also U1.15; no longer U1.27
Routing:
- net GND: track 289.7 -> 287.0 mm
- net LED: track 2.27 -> 4.41 mm
Changed lines of the file:
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@@
 </layers>
 <board>
-<fusionsync huburn="a.cGVyc29uYWw6dWUyYmE2M2My" projecturn="a.cGVyc29uYWw6dWUyYmE2M2MyIzIwMTgwOTE3MTQ5MTY5Mjgx" f3durn="urn:adsk.wipprod:dm.lineage:L9eK_ihpRhugibgrTDCzIw" pcbguid="5a4216a9-1d49-4e33-b541-c1ea75e6242c" lastpulledtime="" lastsyncedchangeguid="4692aed5-cdd3-0a5e-46f1-0a19fefaeb82"/>
+<fusionsync huburn="a.cGVyc29uYWw6dWUyYmE2M2My" projecturn="a.cGVyc29uYWw6dWUyYmE2M2MyIzIwMTgwOTE3MTQ5MTY5Mjgx" f3durn="urn:adsk.wipprod:dm.lineage:L9eK_ihpRhugibgrTDCzIw" pcbguid="5a4216a9-1d49-4e33-b541-c1ea75e6242c" lastpulledtime="" lastsyncedchangeguid="0fada487-5e2e-8cb9-6da7-27cd7fc10aff"/>
 <plain>
 <wire x1="0" y1="0" x2="27.6" y2="0" width="0" layer="20"/>
@@
 <attribute name="VALUE" x="17.78" y="18.669" size="0.762" layer="27" font="vector" align="bottom-center"/>
 </element>
-<element name="J1" library="Molex - 48037-0001" library_urn="urn:adsk.eagle:library:8949197" package="MOLEX_48037-0001_1" package3d_urn="urn:adsk.eagle:package:8949201/2" value="MOLEX_48037-0001" x="13.8" y="-5.588" smashed="yes">
+<element name="J1" library="Molex-48037-0001" library_urn="urn:adsk.eagle:library:9157828" package="MOLEX_48037-0001_1" package3d_urn="urn:adsk.eagle:package:9157833/2" value="MOLEX_48037-0001" x="13.8" y="-5.588" smashed="yes">
 <attribute name="NAME" x="13.192" y="1.348" size="1.016" layer="25" font="vector"/>
 </element>
@@
 <attribute name="VALUE" x="16.383" y="32.385" size="0.762" layer="27" font="vector" rot="R180" align="bottom-center"/>
 </element>
-<element name="LED1" library="gen-discrete" library_urn="urn:adsk.eagle:library:5494231" package="LED1608" package3d_urn="urn:adsk.eagle:package:5494251/3" value="OSBL1608C1A" x="18.542" y="8.89" smashed="yes" rot="R90">
-<attribute name="NAME" x="20.559" y="8.471" size="0.762" layer="25" font="vector" align="bottom-center"/>
-<attribute name="VALUE" x="20.242" y="8.09" size="1.016" layer="27" font="vector" rot="R90"/>
+<element name="LED1" library="gen-discrete" library_urn="urn:adsk.eagle:library:5494231" package="LED1608" package3d_urn="urn:adsk.eagle:package:5494251/3" value="OSBL1608C1A" x="2.794" y="17.907" smashed="yes" rot="R270">
+<attribute name="NAME" x="2.809" y="20.485" size="0.762" layer="25" font="vector" rot="R180" align="bottom-center"/>
+<attribute name="VALUE" x="1.094" y="18.707" size="1.016" layer="27" font="vector" rot="R270"/>
 </element>
 <element name="R1" library="gen-discrete3" library_urn="urn:adsk.eagle:library:8961849" package="RCL_R0402_HS" package3d_urn="urn:adsk.eagle:package:8961860/2" value="10k" x="6.477" y="8.255" smashed="yes" rot="R90">
@@
 <attribute name="VALUE" x="3.048" y="23.876" size="0.762" layer="27" font="vector" align="bottom-center"/>
 </element>
-<element name="R3" library="gen-discrete3" library_urn="urn:adsk.eagle:library:8961849" package="RCL_R0402_HS" package3d_urn="urn:adsk.eagle:package:8961860/2" value="100" x="17.145" y="8.89" smashed="yes" rot="R90">
-<attribute name="NAME" x="17.145" y="6.858" size="0.762" layer="25" font="vector" align="bottom-center"/>
-<attribute name="VALUE" x="18.542" y="8.89" size="0.762" layer="27" font="vector" rot="R90" align="bottom-center"/>
+<element name="R3" library="gen-discrete3" library_urn="urn:adsk.eagle:library:8961849" package="RCL_R0402_HS" package3d_urn="urn:adsk.eagle:package:8961860/2" value="100" x="4.318" y="17.907" smashed="yes" rot="R270">
+<attribute name="NAME" x="5.461" y="18.161" size="0.762" layer="25" font="vector" rot="R180" align="bottom-center"/>
+<attribute name="VALUE" x="2.921" y="17.907" size="0.762" layer="27" font="vector" rot="R270" align="bottom-center"/>
 </element>
 <element name="SW1" library="SKRPACE010" library_urn="urn:adsk.eagle:library:5505983" package="SMT(4.2X3.2)" package3d_urn="urn:adsk.eagle:package:5505988/2" value="SKRPACE010" x="3.81" y="6.35" smashed="yes" rot="R270">
@@
 <wire x1="18.33" y1="21.209" x2="18.33" y2="20.066" width="0.5" layer="1"/>
 <wire x1="18.33" y1="20.066" x2="18.33" y2="18.923" width="0.5" layer="1"/>
-<wire x1="18.542" y1="9.765" x2="19.939" y2="11.162" width="0.5" layer="1"/>
-<wire x1="19.939" y1="11.162" x2="19.939" y2="13.42" width="0.5" layer="1"/>
 <wire x1="17.897234375" y1="12.7325625" x2="19.2515625" y2="12.7325625" width="0.5" layer="1"/>
 <wire x1="19.2515625" y1="12.7325625" x2="19.939" y2="13.42" width="0.5" layer="1"/>
@@
 <wire x1="20.44631875" y1="22.3424" x2="21.37968125" y2="22.3424" width="0.5" layer="1"/>
 <wire x1="20.2106" y1="21.4806" x2="20.2106" y2="22.10668125" width="0.5" layer="1"/>
-<wire x1="1.27" y1="12.319" x2="1.27" y2="22.225" width="0.5" layer="1"/>
+<wire x1="1.27" y1="12.319" x2="1.27" y2="17.145" width="0.5" layer="1"/>
+<wire x1="1.27" y1="17.145" x2="1.27" y2="22.225" width="0.5" layer="1"/>
 <wire x1="1.27" y1="22.225" x2="1.27" y2="24.13" width="0.5" layer="1"/>
 <wire x1="1.27" y1="24.13" x2="1.27" y2="25.273" width="0.5" layer="1"/>
@@
 <wire x1="20.449" y1="1.863" x2="21.844" y2="1.863" width="0.5" layer="1"/>
 <wire x1="10.668" y1="22.606" x2="26.035" y2="22.606" width="0.5" layer="16"/>
+<wire x1="2.794" y1="17.032" x2="1.383" y2="17.032" width="0.5" layer="1"/>
+<wire x1="1.383" y1="17.032" x2="1.27" y2="17.145" width="0.5" layer="1"/>
 </signal>
 <signal name="+3V3" class="2">
@@
 </signal>
 <signal name="LED">
-<contactref element="U1" pad="27"/>
 <contactref element="R3" pad="2"/>
-<wire x1="15.06880625" y1="9.904134375" x2="15.532940625" y2="9.44" width="0.2" layer="1"/>
-<wire x1="15.532940625" y1="9.44" x2="17.145" y2="9.44" width="0.2" layer="1"/>
+<contactref element="U1" pad="15"/>
+<wire x1="8.06845" y1="15.773121875" x2="6.484571875" y2="17.357" width="0.2" layer="1"/>
+<wire x1="6.484571875" y1="17.357" x2="4.318" y2="17.357" width="0.2" layer="1"/>
 </signal>
 <signal name="XOSC1">
@@
 <contactref element="R3" pad="1"/>
 <contactref element="LED1" pad="A"/>
-<wire x1="17.145" y1="8.34" x2="17.47" y2="8.015" width="0.2" layer="1"/>
-<wire x1="17.47" y1="8.015" x2="18.542" y2="8.015" width="0.2" layer="1"/>
+<wire x1="4.318" y1="18.457" x2="3.993" y2="18.782" width="0.2" layer="1"/>
+<wire x1="3.993" y1="18.782" x2="2.794" y2="18.782" width="0.2" layer="1"/>
 </signal>
 </signals>

Commit message: minor update
Parts:
- moved J2 24.0 mm to (2.16, 8.00), turned to 90 degrees
- moved SW1 19.5 mm to (23.1, 8.89), turned to 0 degrees
- moved R1 16.9 mm to (23.1, 11.4), turned to 180 degrees
- moved C2 0.63 mm to (25.5, 4.19)
- moved U3 0.51 mm to (23.0, 4.19)
- moved C1 0.38 mm to (21.5, 2.41)
Routing:
- net GND: track 287.0 -> 322.3 mm
- net SWDIO: track 19.4 -> 9.82 mm
- net BOOT0: track 14.9 -> 6.75 mm, vias 2 -> 0
- net SWCLK: track 18.9 -> 11.2 mm
- net +3V3: track 94.5 -> 90.1 mm, vias 7 -> 8
- net NRST: track 17.9 -> 21.5 mm, vias 2 -> 0
- net USB_D-: track 10.7 -> 9.35 mm
- net USB_D+: track 6.32 -> 7.34 mm
- net +5V: track 7.20 -> 6.64 mm
Other:
- board text added: "GND"
- board text added: "NRST"
- board text added: "SWCLK"
- board text added: "SWDIO"
